Commit message: Hexabot first training run

File: hexabot_model/isaac/hexabot.urdf (robot description, URDF)
Before this commit: robot hexabot, 19 links, 18 joints
Joints:
- joint tibia_lf: limit lower=-1.5500 upper=0.4500 effort=1.08 velocity=6.16 -> lower=-1.5500 upper=1.4000 effort=1.08 velocity=6.16
- joint tibia_lm: limit lower=-1.5500 upper=0.4500 effort=1.08 velocity=6.16 -> lower=-1.5500 upper=1.4000 effort=1.08 velocity=6.16
- joint tibia_lr: limit lower=-1.5500 upper=0.4500 effort=1.08 velocity=6.16 -> lower=-1.5500 upper=1.4000 effort=1.08 velocity=6.16
- joint tibia_rf: limit lower=-1.5500 upper=0.4500 effort=1.08 velocity=6.16 -> lower=-1.5500 upper=1.4000 effort=1.08 velocity=6.16
- joint tibia_rm: limit lower=-1.5500 upper=0.4500 effort=1.08 velocity=6.16 -> lower=-1.5500 upper=1.4000 effort=1.08 velocity=6.16
- joint tibia_rr: limit lower=-1.5500 upper=0.4500 effort=1.08 velocity=6.16 -> lower=-1.5500 upper=1.4000 effort=1.08 velocity=6.16
